File: a8sram.kicad_pcb (KiCad board)
At the start: 2 copper layers, 8 parts, among them J1 D, U1 GAL16V8, U5 KM62256CLP, U6 KM62256CLP

Commit message: wip
Connections:
- net _CE1 renamed _OE1
- net _CE2 renamed _OE2
- U1 pad 11: unconnected-(U1-I10/~{OE}-Pad11) -> GND
- U1 pad 9: unconnected-(U1-I9-Pad9) -> A15
Routing:
- net A15: track 0.00 -> 50.6 mm
- net GND: track 133.1 -> 121.6 mm, vias 0 -> 4
- net RW: track 77.1 -> 76.2 mm
- added copper zone on B.Cu, net GND
- added copper zone on F.Cu, net GND
Other:
- board outline added: 45 x 55 mm
