File: 2x32k-gal/a8sram.kicad_pcb (KiCad board)
At the start: 2 copper layers, 45 x 55 mm, 10 parts, among them J1 D, U1 GAL16V8, U5 KM62256CLP, U6 KM62256CLP

Commit message: Cleanup.
Connections:
- U1 pad 6: I6 -> unconnected-(U1-I6-Pad6)
- U1 pad 7: I7 -> unconnected-(U1-I7-Pad7)
- U1 pad 8: I8 -> unconnected-(U1-I8-Pad8)
Changed lines of the file:
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@@
 	(net 44 "unconnected-(U4-NC-Pad36)")
 	(net 45 "unconnected-(U4-RA5-Pad27)")
-	(net 46 "I8")
+	(net 46 "unconnected-(U1-I6-Pad6)")
 	(net 47 "CLK{slash}2")
 	(net 48 "O5")
 	(net 49 "O4")
-	(net 50 "I7")
-	(net 51 "I6")
+	(net 50 "unconnected-(U1-I7-Pad7)")
+	(net 51 "unconnected-(U1-I8-Pad8)")
 	(net 52 "O3")
 	(net 53 "Net-(JP1-C)")
@@
 			(layers "*.Cu" "*.Mask")
 			(remove_unused_layers no)
-			(net 51 "I6")
+			(net 46 "unconnected-(U1-I6-Pad6)")
 			(pinfunction "I6")
-			(pintype "input")
+			(pintype "input+no_connect")
 		)
 		(pad "7" thru_hole circle
@@
 			(layers "*.Cu" "*.Mask")
 			(remove_unused_layers no)
-			(net 50 "I7")
+			(net 50 "unconnected-(U1-I7-Pad7)")
 			(pinfunction "I7")
-			(pintype "input")
+			(pintype "input+no_connect")
 		)
 		(pad "8" thru_hole circle
@@
 			(layers "*.Cu" "*.Mask")
 			(remove_unused_layers no)
-			(net 46 "I8")
+			(net 51 "unconnected-(U1-I8-Pad8)")
 			(pinfunction "I8")
-			(pintype "input")
+			(pintype "input+no_connect")
 		)
 		(pad "9" thru_hole circle
